Commit message: update readme and some parameters in cfg

File: assets/urdf/aliengo/urdf/aliengo.urdf (robot description, URDF)
Before this commit: robot aliengo_description, 17 links, 16 joints
Joints:
- joint FL_thigh_joint: limit effort=44.4 velocity=40 -> lower=-1.570795 upper=1.570795 effort=44.4 velocity=40
- joint FR_thigh_joint: limit effort=44.4 velocity=40 -> lower=-1.570795 upper=1.570795 effort=44.4 velocity=40
- joint RL_thigh_joint: limit effort=44.4 velocity=40 -> lower=-1.570795 upper=1.570795 effort=44.4 velocity=40
- joint RR_thigh_joint: limit effort=44.4 velocity=40 -> lower=-1.570795 upper=1.570795 effort=44.4 velocity=40
